File: PCB/PCB Shield/Mega_2560 core mini_full_2.2_PM/OpenAVRc_CoreConnects.sch (KiCad schematic (older format))
At the start: 24 parts, among them P1 2560-core, P10 RX1TX1, P15 Micro_sd, P16 LCD, P6 SPI, P9 DUMMY, Q1 IRLML5203

Commit message: Add SCC feature for SBUS servo programmation
Parts:
- added P27: SCC, Mylib_v2.2:Pin_Header_Straight_1x03_Pitch2.54mm, symbol Mega_2560-core-mini_full_2.2-rescue:CONN_01X03-Mega_2560-core-mini_full_2.1-Meg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
- added R47: 100K, Mylib_v2.2:R_1206, symbol Mega_2560-core-mini_full_2.2-rescue:R-RESCUE-Mega_2560_core_mini_full_2.0-Mega_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
- added R48: 1K, Mylib_v2.2:R_1206, symbol Mega_2560-core-mini_full_2.2-rescue:R-RESCUE-Mega_2560_core_mini_full_2.0-Mega_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
- C18, C3: footprint Capacitors_SMD:C_1206 -> Mylib_v2.2:C_1206
Connections:
- net GND: now also P27.3 (P3), R47.2
- net VCC: now also P27.2 (P2)
- net SCC: now reaches P1.J2 (P59)
- net SCC: now also R48.2
- new net: P27.1 (P1), R47.1, R48.1
- no-connect marks 4 -> 3
Other:
- moved on the sheet: P16, R40, RV1, RV6
